File: Anzeigeplatine/pcb/Messwagen Anzeigeplatine.kicad_pcb (KiCad board)
At the start: 2 copper layers, 86.7 x 24.1 mm, 68 parts, among them IC1 MAX7219CWG, J1 Conn_01x05, U1 HDSP-7503, U2 HDSP-7503, U3 HDSP-7503, U4 HDSP-7503

Commit message: Add files via upload
Parts:
- C1, R1: moved to B.Cu
- moved J1 9.68 mm to (35.7, 31.6)
- moved C1 7.11 mm to (41.7, 32.5), turned to 90 degrees
- moved R1 4.11 mm to (39.3, 32.5), turned to 270 degrees
Routing:
- net +5V: track 21.2 -> 12.3 mm
- net GND: track 0.00 -> 7.79 mm, vias 6 -> 10
- net Net-(IC1-Pad18): track 8.59 -> 2.97 mm, vias 1 -> 0
- net /LOAD: track 10.9 -> 14.8 mm
- net /CLK: track 11.8 -> 8.98 mm
- net /D_IN: track 14.6 -> 12.5 mm
- net /PC: track 69.0 -> 70.3 mm
