File: Neigungsmesswagen/pcb/Neigungsmesswagen.kicad_pcb (KiCad board)
At the start: 2 copper layers, 79.8 x 24.9 mm, 45 parts, among them IC1 D_Bridge, IC2 TSR_1-2450, IC3 ATmega328, IC4 6N137, IC5 ULN2003, J1 ISP, J2 Display, Q1 16MHz

Commit message: Add files via upload
Parts:
- added CC-Logo1: ---, Symbol:CC-BY-NC-SA_10x3.6mm_SilkScreen, B.Cu at (25.3, 22.4)
