File: Neigungsmesswagen/pcb/Neigungsmesswagen.sch (KiCad schematic (older format))
At the start: 45 parts, among them IC1 D_Bridge, IC2 TSR_1-2450, IC3 ATmega328, IC4 6N137, IC5 ULN2003, J1 ISP, J2 Display, Q1 16MHz

Commit message: Add files via upload
Parts:
- added CC-Logo1: ---, Symbol:CC-BY-NC-SA_10x3.6mm_SilkScreen, symbol Mechanical:MountingHole
Changed lines of the file:
@@
 	9600 5800 9850 5800
 Connection ~ 9850 5800
+$Comp
+L Mechanical:MountingHole CC-Logo1
+U 1 1 5E718CE6
+P 550 950
+F 0 "CC-Logo1" H 650 950 50  0000 L CNN
+F 1 "---" H 650 905 50  0001 L CNN
+F 2 "Symbol:CC-BY-NC-SA_10x3.6mm_SilkScreen" H 550 950 50  0001 C CNN
+F 3 "---" H 550 950 50  0001 C CNN
+F 4 "---" H -100 0   50  0001 C CNN "Lieferant"
+F 5 "---" H -100 0   50  0001 C CNN "Nummer"
+F 6 "---" H 0   200 50  0001 C CNN "Vorrätig"
+	1    550  950
+	1    0    0    -1
+$EndComp
 $EndSCHEMATC
